File: pcb/board2.kicad_pcb (KiCad board)
At the start: 4 copper layers, 48.5 x 44.5 mm, 29 parts, among them J1 Conn_01x04_Socket, J2 Conn_01x02_Socket, J3 Conn_01x02_Socket, J4 Conn_01x03_Socket, J5 Conn_01x02_Socket, J7 Conn_01x03_Socket, Q1 AO3400A, SW1 TS-1101-B-W, SW3 TS-1101-B-W, U1 AMS1117-5.0, U19 ESP32-WROOM-32, U20 SPX3819M5-L-3-3

Commit message: CODE
Parts:
- moved R2 4.83 mm to (205.0, 114.2)
Routing:
- net /3.3v_esp: track 12.4 -> 79.5 mm, vias 6 -> 7
- net Net-(U19-IO0): track 34.5 -> 51.4 mm, vias 4 -> 0
- net Net-(J4-Pin_2): track 63.6 -> 56.9 mm
- net /B+: track 99.7 -> 96.7 mm
- net Net-(U19-IO17): track 60.6 -> 63.1 mm, vias 2 -> 0
- net /BVOL: track 38.5 -> 40.8 mm
- net Net-(U19-EN): track 20.3 -> 21.4 mm
- removed copper zone on In2.Cu, net /3.3v_esp
- removed copper zone on In1.Cu, net GND
Other:
- copper layers 4 -> 2
