File: pcb/board2.kicad_sch (KiCad schematic)
At the start: 29 parts, among them J1 Conn_01x04_Socket, J2 Conn_01x02_Socket, J3 Conn_01x02_Socket, J4 Conn_01x03_Socket, J5 Conn_01x02_Socket, J7 Conn_01x03_Socket, Q1 AO3400A, SW1 TS-1101-B-W, SW3 TS-1101-B-W, U1 AMS1117-5.0, U19 ESP32-WROOM-32, U20 SPX3819M5-L-3-3

Commit message: CODE
Other:
- note added: "button input"
- note added: "fan port"
- moved on the sheet: J1, J2, J4, J7, Q1, R1, R2
